Commit message: v2: improved IK stability, added rosbridge + web interface, fixed URDF alignment

File: install/dof6arm/share/dof6arm/urdf/dof6arm.urdf (robot description, URDF)
Before this commit: robot dof6arm, 8 links, 7 joints
Links:
- added link world_rviz
Joints:
- added joint world_joint: type fixed, parent world_rviz, child base_link, origin xyz=0 0 0 rpy=0 0 -1.5708
