Commit message: clude preaynsh 1.0 corrected minor mistakes and added gazebo but with unit of mm 9 may 26'

File: src/dof6arm/urdf/backup.urdf (robot description, URDF)
Before this commit: robot dof6arm, 8 links, 7 joints
Links:
- added link world
- link base_link: mass 5.51043299491621 -> 5.5104; geometry collision box size=0.3 0.3 0.1; visual mesh filename=package://dof6arm/meshes/base_link.STL
- link endfector: mass 0.0762574810565132 -> None; geometry collision box size=0.1 0.1 0.1; visual mesh filename=package://dof6arm/meshes/endfector.STL
- link link1: mass 2.25493378297323 -> 2.2; geometry collision box size=0.2 0.2 0.3; visual mesh filename=package://dof6arm/meshes/link1.STL
- link link2: mass 0.920714229759599 -> 0.9; geometry collision box size=0.2 0.4 0.1; visual mesh filename=package://dof6arm/meshes/link2.STL
- link link3: mass 1.43145554418529 -> None; geometry collision box size=0.2 0.2 0.2; visual mesh filename=package://dof6arm/meshes/link3.STL
- link link4: mass 0.581435273248316 -> None; geometry collision box size=0.2 0.2 0.2; visual mesh filename=package://dof6arm/meshes/link4.STL
- link link5: mass 0.339144547925522 -> None; geometry collision box size=0.15 0.15 0.2; visual mesh filename=package://dof6arm/meshes/link5.STL
- link link6: mass 0.0762574810565132 -> None; geometry collision box size=0.1 0.1 0.1; visual mesh filename=package://dof6arm/meshes/link6.STL
Joints:
- removed joint joint0
- added joint joint7: type fixed, parent link6, child endfector, origin xyz=0 0 0.045
- added joint world_fixed: type fixed, parent world, child base_link
- joint joint1: child link2 -> link1; limit lower=-0.70 upper=0.70 effort=200 velocity=10 -> lower=-3.14 upper=3.14 effort=20 velocity=10; origin xyz=0.150000000000022 -0.019999999999832 0.159999999999999 rpy=1.5707963267949 0 0 -> xyz=0 0 0.085 rpy=0 0 1.5708; parent link1 -> base_link; type continuous -> revolute
- joint joint2: child link3 -> link2; limit lower=-4.71 upper=1.57 effort=200 velocity=10 -> lower=-1.57 upper=1.57 effort=20 velocity=10; origin xyz=0 0.350000000000001 0 rpy=0 0 1.5707963267949 -> xyz=0.15 -0.02 0.16 rpy=1.5708 0 0; parent link2 -> link1; type continuous -> revolute
- joint joint3: child link4 -> link3; limit lower=-3.14 upper=3.14 effort=200 velocity=10 -> lower=-1.57 upper=1.57 effort=20 velocity=10; origin xyz=-0.045 -0.251 -0.0474999999999995 rpy=1.5707963267949 0 0 -> xyz=0 0.35 0 rpy=0 0 1.5708; parent link3 -> link2; type continuous -> revolute
- joint joint4: child link5 -> link4; limit lower=-1.57 upper=1.57 effort=200 velocity=10 -> lower=-1.57 upper=1.57 effort=20 velocity=10; origin xyz=0 0.00050000000000075 0.11 rpy=-1.5707963267949 0 0 -> xyz=-0.045 -0.251 -0.0475 rpy=1.5708 0 0; parent link4 -> link3; type continuous -> revolute
- joint joint5: child link6 -> link5; limit lower=-3.14 upper=3.14 effort=200 velocity=10 -> lower=-1.57 upper=1.57 effort=20 velocity=10; origin xyz=0 -0.104 0 rpy=1.5707963267949 0 0 -> xyz=0 0.0005 0.11 rpy=-1.5708 0 0; parent link5 -> link4; type continuous -> revolute
- joint joint6: axis 0 0 0 -> 0 0 1; child endfector -> link6; limit (none) -> lower=-1.57 upper=1.57 effort=20 velocity=10; origin xyz=0 0 0.045605 rpy=0 0 0 -> xyz=0 -0.104 0 rpy=1.5708 0 0; parent link6 -> link5; type fixed -> revolute
