Commit message: calude v2.0 gazebo with added tip as EE

File: src/dof6arm/urdf/dof6arm_gazebo.urdf.xacro (robot description, xacro)
@@ -1,4 +1,4 @@
 <robot xmlns:xacro="http://www.ros.org/wiki/xacro" name="dof6arm">
-  <link name="world"/>
+  <!-- <link name="world"/>
   <link
     name="base_link">
@@ -452,4 +452,457 @@
     <axis
       xyz="0 0 0" />
+  </joint> -->
+  <link name="world"/>
+  <link
+    name="base_link">
+    <inertial>
+      <origin
+        xyz="-2.8338E-17 -1.0375E-17 0.039627"
+        rpy="0 0 0" />
+      <mass
+        value="5.5104" />
+      <inertia
+        ixx="0.032533"
+        ixy="-5.7178E-17"
+        ixz="1.4037E-17"
+        iyy="0.032533"
+        iyz="-4.4371E-17"
+        izz="0.058905" />
+    </inertial>
+    <visual>
+      <origin
+        xyz="0 0 0"
+        rpy="0 0 0" />
+      <geometry>
+        <mesh
+          filename="package://dof6arm/meshes/base_link.STL" />
+      </geometry>
+      <material
+        name="">
+        <color
+          rgba="0.058824 0.058824 0.058824 1" />
+      </material>
+    </visual>
+    <collision>
+      <origin
+        xyz="0 0 0"
+        rpy="0 0 0" />
+      <geometry>
+        <mesh
+          filename="package://dof6arm/meshes/base_link.STL" />
+      </geometry>
+    </collision>
+  </link>
+  <joint name="world_joint" type="fixed">
+    <parent link="world"/>
+    <child link="base_link"/>
+    <origin xyz="0 0 0" rpy="0 0 -1.5708"/>
+  </joint>
+  <link
+    name="link1">
+    <inertial>
+      <origin
+        xyz="0.056315 0.0023965 0.081396"
+        rpy="0 0 0" />
+      <mass
+        value="2.2549" />
+      <inertia
+        ixx="0.011608"
+        ixy="-0.00040169"
+        ixz="-0.0088797"
+        iyy="0.023156"
+        iyz="-0.00035105"
+        izz="0.01588" />
+    </inertial>
+    <visual>
+      <origin
+        xyz="0 0 0"
+        rpy="0 0 0" />
+      <geometry>
+        <mesh
+          filename="package://dof6arm/meshes/link1.STL" />
+      </geometry>
+      <material
+        name="">
+        <color
+          rgba="0.89804 0.91765 0.92941 1" />
+      </material>
+    </visual>
+    <collision>
+      <origin
+        xyz="0 0 0"
+        rpy="0 0 0" />
+      <geometry>
+        <mesh
+          filename="package://dof6arm/meshes/link1.STL" />
+      </geometry>
+    </collision>
+  </link>
+  <joint
+    name="joint1"
+    type="revolute">
+    <origin
+      xyz="0 0 0.085"
+      rpy="0 0 1.5708" />
+    <parent
+      link="base_link" />
+    <child
+      link="link1" />
+    <axis
+      xyz="0 0 1" />
+    <limit
+      lower="-3.14"
+      upper="3.14"
+      effort="2000"
+      velocity="10" />
+      <dynamics damping="5.0" friction="0.5"/>
+  </joint>
+  <link
+    name="link2">
+    <inertial>
+      <origin
+        xyz="-0.0080603 0.14266 0.015223"
+        rpy="0 0 0" />
+      <mass
+        value="0.92071" />
+      <inertia
+        ixx="0.017861"
+        ixy="0.00015241"
+        ixz="-3.0375E-05"
+        iyy="0.00061487"
+        iyz="7.163E-05"
+        izz="0.018205" />
+    </inertial>
+    <visual>
+      <origin
+        xyz="0 0 0"
+        rpy="0 0 0" />
+      <geometry>
+        <mesh
+          filename="package://dof6arm/meshes/link2.STL" />
+      </geometry>
+      <material
+        name="">
+        <color
+          rgba="0.63922 0.66667 0.67843 1" />
+      </material>
+    </visual>
+    <collision>
+      <origin
+        xyz="0 0 0"
+        rpy="0 0 0" />
+      <geometry>
+        <mesh
+          filename="package://dof6arm/meshes/link2.STL" />
+      </geometry>
+    </collision>
+  </link>
+  <joint
+    name="joint2"
+    type="revolute">
+    <origin
+      xyz="0.15 -0.02 0.16"
+      rpy="1.5708 0 0" />
+    <parent
+      link="link1" />
+    <child
+      link="link2" />
+    <axis
+      xyz="0 0 1" />
+    <limit
+      lower="-1.57"
+      upper="1.57"
+      effort="2000"
+      velocity="10" />
+      <dynamics damping="5.0" friction="0.5"/>
+  </joint>
+  <link
+    name="link3">
+    <inertial>
+      <origin
+        xyz="-0.037874 -0.081929 -0.0086553"
+        rpy="0 0 0" />
+      <mass
+        value="1.4315" />
+      <inertia
+        ixx="0.0080768"
+        ixy="-0.00032475"
+        ixz="-0.00011286"
+        iyy="0.0018664"
+        iyz="-9.3414E-05"
+        izz="0.0084455" />
+    </inertial>
+    <visual>
+      <origin
+        xyz="0 0 0"
+        rpy="0 0 0" />
+      <geometry>
+        <mesh
+          filename="package://dof6arm/meshes/link3.STL" />
+      </geometry>
+      <material
+        name="">
+        <color
+          rgba="0.89804 0.91765 0.92941 1" />
+      </material>
+    </visual>
+    <collision>
+      <origin
+        xyz="0 0 0"
+        rpy="0 0 0" />
+      <geometry>
+        <mesh
+          filename="package://dof6arm/meshes/link3.STL" />
+      </geometry>
+    </collision>
+  </link>
+  <joint
+    name="joint3"
+    type="revolute">
+    <origin
+      xyz="-0.0373120803311945 0.347958550658273 -0.0373820601117326"
+      rpy="0 0 1.5707963267949" />
+    <parent
+      link="link2" />
+    <child
+      link="link3" />
+    <axis
+      xyz="0 0 1" />
+    <limit
+      lower="-3.14"
+      upper="1.57"
+      effort="2000"
+      velocity="10" />
+      <dynamics damping="5.0" friction="0.5"/>
+  </joint>
+  <link
+    name="link4">
+    <inertial>
+      <origin
+        xyz="0 1.38777878078145E-17 0.0659648893354512"
+        rpy="0 0 0" />
+      <mass
+        value="0.581435273248316" />
+      <inertia
+        ixx="0.00158017066215487"
+        ixy="2.44381629744968E-10"
+        ixz="-4.57912642337429E-19"
+        iyy="0.0014063460239573"
+        iyz="-2.68731603937658E-19"
+        izz="0.000596523986913167" />
+    </inertial>
+    <visual>
+      <origin
+        xyz="0 0 0"
+        rpy="0 0 0" />
+      <geometry>
+        <mesh
+          filename="package://dof6arm/meshes/link4.STL" />
+      </geometry>
+      <material
+        name="">
+        <color
+          rgba="0.792156862745098 0.819607843137255 0.933333333333333 1" />
+      </material>
+    </visual>
+    <collision>
+      <origin
+        xyz="0 0 0"
+        rpy="0 0 0" />
+      <geometry>
+        <mesh
+          filename="package://dof6arm/meshes/link4.STL" />
+      </geometry>
+    </collision>
+  </link>
+  <joint
+    name="joint4"
+    type="revolute">
+    <origin
+      xyz="-0.0429585506582734 -0.288312080331216 -0.0101179398882675"
+      rpy="1.5707963267949 0 0" />
+    <parent
+      link="link3" />
+    <child
+      link="link4" />
+    <axis
+      xyz="0 0 1" />
+    <limit
+      lower="-3.14"
+      upper="3.14"
+      effort="2000"
+      velocity="10" />
+  </joint>
+  <link
+    name="link5">
+    <inertial>
+      <origin
+        xyz="-2.22044604925031E-16 -0.0589618551288013 0.000178318239085751"
+        rpy="0 0 0" />
+      <mass
+        value="0.339144547925523" />
+      <inertia
+        ixx="0.000355541202477726"
+        ixy="9.17440418306188E-21"
+        ixz="-3.40456917885845E-21"
+        iyy="0.000248853470602005"
+        iyz="-3.56575702010602E-06"
+        izz="0.000358769992191288" />
+    </inertial>
+    <visual>
+      <origin
+        xyz="0 0 0"
+        rpy="0 0 0" />
+      <geometry>
+        <mesh
+          filename="package://dof6arm/meshes/link5.STL" />
+      </geometry>
+      <material
+        name="">
+        <color
+          rgba="0.898039215686275 0.917647058823529 0.929411764705882 1" />
+      </material>
+    </visual>
+    <collision>
+      <origin
+        xyz="0 0 0"
+        rpy="0 0 0" />
+      <geometry>
+        <mesh
+          filename="package://dof6arm/meshes/link5.STL" />
+      </geometry>
+    </collision>
+  </link>
+  <joint
+    name="joint5"
+    type="revolute">
+    <origin
+      xyz="0 0.000499999999999997 0.109999999999978"
+      rpy="-1.5707963267949 0 0" />
+    <parent
+      link="link4" />
+    <child
+      link="link5" />
+    <axis
+      xyz="0 0 1" />
+    <limit
+      lower="-1.57"
+      upper="1.57"
+      effort="2000"
+      velocity="10" />
+      <dynamics damping="5.0" friction="0.5"/>
+  </joint>
+  <link
+    name="link6">
+    <inertial>
+      <origin
+        xyz="0 0 0.00628470620704236"
+        rpy="0 0 0" />
+      <mass
+        value="0.0762574810565132" />
+      <inertia
+        ixx="3.79559798700621E-05"
+        ixy="1.86509367076551E-21"
+        ixz="-6.62000777514621E-22"
+        iyy="3.20288004196063E-05"
+        iyz="1.93589180543697E-21"
+        izz="3.99525744954329E-05" />
+    </inertial>
+    <visual>
+      <origin
+        xyz="0 0 0"
+        rpy="0 0 0" />
+      <geometry>
+        <mesh
+          filename="package://dof6arm/meshes/link6.STL" />
+      </geometry>
+      <material
+        name="">
+        <color
+          rgba="0.898039215686275 0.917647058823529 0.929411764705882 1" />
+      </material>
+    </visual>
+    <collision>
+      <origin
+        xyz="0 0 0"
+        rpy="0 0 0" />
+      <geometry>
+        <mesh
+          filename="package://dof6arm/meshes/link6.STL" />
+      </geometry>
+    </collision>
+  </link>
+  <joint
+    name="joint6"
+    type="revolute">
+    <origin
+      xyz="0 -0.104 0"
+      rpy="1.5708 0 0" />
+    <parent
+      link="link5" />
+    <child
+      link="link6" />
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